Commit message: Push updates, still need to fix minimum distance constraint deprecation fix

File: examples/scora/models/movable_box_point.urdf (robot description, URDF)
Before this commit: robot box, 3 links, 3 joints
Links:
- link box_link_1: geometry collision box size=0.01 0.01 0.01; visual box size=0.05 0.05 0.05
